Commit message: Checkpoint

File: src/forklift_description_realistic/urdf/rear_steer_forklift.urdf.xacro (robot description, xacro)
@@ -8,4 +8,6 @@
   <xacro:property name="front_track" value="0.92"/>
   <xacro:property name="rear_track" value="0.78"/>
+  <xacro:property name="ground_clearance" value="0.08"/>
+  <xacro:property name="body_base_z" value="${ground_clearance}"/>
   <xacro:property name="chassis_length" value="1.80"/>
   <xacro:property name="chassis_width" value="1.10"/>
@@ -24,10 +26,19 @@
   <xacro:property name="fork_height" value="0.05"/>
   <xacro:property name="fork_gap" value="0.82"/>
-  <xacro:property name="roof_z" value="${wheel_radius + chassis_height + cabin_height}"/>
+  <xacro:property name="roof_z" value="${body_base_z + chassis_height + cabin_height}"/>
   <xacro:property name="mast_x" value="0.98"/>
-  <link name="base_link"/>
-  <link name="chassis_link">
-    <visual>
-      <origin xyz="0 0 ${wheel_radius + chassis_height / 2.0}"/>
+  <xacro:property name="rear_steer_link_center_z" value="${wheel_radius + 0.05}"/>
+  <xacro:property name="counterweight_length" value="0.42"/>
+  <xacro:property name="counterweight_width" value="1.00"/>
+  <xacro:property name="counterweight_height" value="0.72"/>
+  <xacro:property name="counterweight_x" value="-0.62"/>
+  <xacro:property name="counterweight_z" value="${body_base_z + counterweight_height / 2.0}"/>
+  <xacro:property name="support_skid_length" value="0.80"/>
+  <xacro:property name="support_skid_width" value="0.40"/>
+  <xacro:property name="support_skid_height" value="0.02"/>
+  <xacro:property name="support_skid_z" value="0.16"/>
+  <link name="base_link">
+    <visual>
+      <origin xyz="0 0 ${body_base_z + chassis_height / 2.0}"/>
       <geometry>
         <box size="${chassis_length} ${chassis_width} ${chassis_height}"/>
@@ -38,21 +49,16 @@
     </visual>
     <collision>
-      <origin xyz="0 0 ${wheel_radius + chassis_height / 2.0}"/>
-      <geometry>
-        <box size="${chassis_length} ${chassis_width} ${chassis_height}"/>
-      </geometry>
-    </collision>
-    <xacro:inertial_box mass="950.0" x="${chassis_length}" y="${chassis_width}" z="${chassis_height}">
-      <origin xyz="0 0 ${wheel_radius + chassis_height / 2.0}"/>
-    </xacro:inertial_box>
-  </link>
-  <joint name="base_to_chassis" type="fixed">
-    <parent link="base_link"/>
-    <child link="chassis_link"/>
-    <origin xyz="0 0 0"/>
-  </joint>
+      <origin xyz="0 0 ${support_skid_z}"/>
+      <geometry>
+        <box size="${support_skid_length} ${support_skid_width} ${support_skid_height}"/>
+      </geometry>
+    </collision>
+    <xacro:inertial_box mass="1100.0" x="${chassis_length}" y="${chassis_width}" z="${chassis_height}">
+      <origin xyz="0 0 ${body_base_z + chassis_height / 2.0}"/>
+    </xacro:inertial_box>
+  </link>
   <link name="cabin_link">
     <visual>
-      <origin xyz="-0.10 0 ${wheel_radius + chassis_height + cabin_height / 2.0}"/>
+      <origin xyz="-0.10 0 ${body_base_z + chassis_height + cabin_height / 2.0}"/>
       <geometry>
         <box size="${cabin_length} ${cabin_width} ${cabin_height}"/>
@@ -62,22 +68,37 @@
       </material>
     </visual>
-    <collision>
-      <origin xyz="-0.10 0 ${wheel_radius + chassis_height + cabin_height / 2.0}"/>
-      <geometry>
-        <box size="${cabin_length} ${cabin_width} ${cabin_height}"/>
-      </geometry>
-    </collision>
-    <xacro:inertial_box mass="420.0" x="${cabin_length}" y="${cabin_width}" z="${cabin_height}">
-      <origin xyz="-0.10 0 ${wheel_radius + chassis_height + cabin_height / 2.0}"/>
+    <xacro:inertial_box mass="280.0" x="${cabin_length}" y="${cabin_width}" z="${cabin_height}">
+      <origin xyz="-0.10 0 ${body_base_z + chassis_height + cabin_height / 2.0}"/>
     </xacro:inertial_box>
   </link>
   <joint name="chassis_to_cabin" type="fixed">
-    <parent link="chassis_link"/>
+    <parent link="base_link"/>
     <child link="cabin_link"/>
     <origin xyz="0 0 0"/>
   </joint>
+  <link name="counterweight_link">
+    <visual>
+      <origin xyz="${counterweight_x} 0 ${counterweight_z}"/>
+      <geometry>
+        <box size="${counterweight_length} ${counterweight_width} ${counterweight_height}"/>
+      </geometry>
+      <material name="dark_gray"/>
+    </visual>
+    <xacro:inertial_box
+      mass="680.0"
+      x="${counterweight_length}"
+      y="${counterweight_width}"
+      z="${counterweight_height}">
+      <origin xyz="${counterweight_x} 0 ${counterweight_z}"/>
+    </xacro:inertial_box>
+  </link>
+  <joint name="chassis_to_counterweight" type="fixed">
+    <parent link="base_link"/>
+    <child link="counterweight_link"/>
+    <origin xyz="0 0 0"/>
+  </joint>
   <link name="mast_link">
     <visual>
-      <origin xyz="${mast_x} 0 ${wheel_radius + mast_height / 2.0}"/>
+      <origin xyz="${mast_x} 0 ${body_base_z + mast_height / 2.0}"/>
       <geometry>
         <box size="${mast_depth} ${mast_width} ${mast_height}"/>
@@ -87,16 +108,10 @@
       </material>
     </visual>
-    <collision>
-      <origin xyz="${mast_x} 0 ${wheel_radius + mast_height / 2.0}"/>
-      <geometry>
-        <box size="${mast_depth} ${mast_width} ${mast_height}"/>
-      </geometry>
-    </collision>
-    <xacro:inertial_box mass="260.0" x="${mast_depth}" y="${mast_width}" z="${mast_height}">
-      <origin xyz="${mast_x} 0 ${wheel_radius + mast_height / 2.0}"/>
+    <xacro:inertial_box mass="230.0" x="${mast_depth}" y="${mast_width}" z="${mast_height}">
+      <origin xyz="${mast_x} 0 ${body_base_z + mast_height / 2.0}"/>
     </xacro:inertial_box>
   </link>
   <joint name="chassis_to_mast" type="fixed">
-    <parent link="chassis_link"/>
+    <parent link="base_link"/>
     <child link="mast_link"/>
     <origin xyz="0 0 0"/>
@@ -104,5 +119,5 @@
   <link name="fork_base_link">
     <visual>
-      <origin xyz="${mast_x + carriage_depth / 2.0} 0 ${wheel_radius + carriage_height / 2.0}"/>
+      <origin xyz="${mast_x + carriage_depth / 2.0} 0 ${body_base_z + carriage_height / 2.0}"/>
       <geometry>
         <box size="${carriage_depth} ${carriage_width} ${carriage_height}"/>
@@ -112,12 +127,6 @@
       </material>
     </visual>
-    <collision>
-      <origin xyz="${mast_x + carriage_depth / 2.0} 0 ${wheel_radius + carriage_height / 2.0}"/>
-      <geometry>
-        <box size="${carriage_depth} ${carriage_width} ${carriage_height}"/>
-      </geometry>
-    </collision>
-    <xacro:inertial_box mass="140.0" x="${carriage_depth}" y="${carriage_width}" z="${carriage_height}">
-      <origin xyz="${mast_x + carriage_depth / 2.0} 0 ${wheel_radius + carriage_height / 2.0}"/>
+    <xacro:inertial_box mass="120.0" x="${carriage_depth}" y="${carriage_width}" z="${carriage_height}">
+      <origin xyz="${mast_x + carriage_depth / 2.0} 0 ${body_base_z + carriage_height / 2.0}"/>
     </xacro:inertial_box>
   </link>
@@ -132,5 +141,5 @@
   <link name="left_fork_link">
     <visual>
-      <origin xyz="${mast_x + carriage_depth + fork_length / 2.0} ${fork_gap / 2.0} ${wheel_radius + 0.08}"/>
+      <origin xyz="${mast_x + carriage_depth + fork_length / 2.0} ${fork_gap / 2.0} ${body_base_z + 0.08}"/>
       <geometry>
         <box size="${fork_length} ${fork_width} ${fork_height}"/>
@@ -138,12 +147,6 @@
       <material name="steel"/>
     </visual>
-    <collision>
-      <origin xyz="${mast_x + carriage_depth + fork_length / 2.0} ${fork_gap / 2.0} ${wheel_radius + 0.08}"/>
-      <geometry>
-        <box size="${fork_length} ${fork_width} ${fork_height}"/>
-      </geometry>
-    </collision>
-    <xacro:inertial_box mass="22.0" x="${fork_length}" y="${fork_width}" z="${fork_height}">
-      <origin xyz="${mast_x + carriage_depth + fork_length / 2.0} ${fork_gap / 2.0} ${wheel_radius + 0.08}"/>
+    <xacro:inertial_box mass="18.0" x="${fork_length}" y="${fork_width}" z="${fork_height}">
+      <origin xyz="${mast_x + carriage_depth + fork_length / 2.0} ${fork_gap / 2.0} ${body_base_z + 0.08}"/>
     </xacro:inertial_box>
   </link>
@@ -155,5 +158,5 @@
   <link name="right_fork_link">
     <visual>
-      <origin xyz="${mast_x + carriage_depth + fork_length / 2.0} -${fork_gap / 2.0} ${wheel_radius + 0.08}"/>
+      <origin xyz="${mast_x + carriage_depth + fork_length / 2.0} -${fork_gap / 2.0} ${body_base_z + 0.08}"/>
       <geometry>
         <box size="${fork_length} ${fork_width} ${fork_height}"/>
@@ -161,12 +164,6 @@
       <material name="steel"/>
     </visual>
-    <collision>
-      <origin xyz="${mast_x + carriage_depth + fork_length / 2.0} -${fork_gap / 2.0} ${wheel_radius + 0.08}"/>
-      <geometry>
-        <box size="${fork_length} ${fork_width} ${fork_height}"/>
-      </geometry>
-    </collision>
-    <xacro:inertial_box mass="22.0" x="${fork_length}" y="${fork_width}" z="${fork_height}">
-      <origin xyz="${mast_x + carriage_depth + fork_length / 2.0} -${fork_gap / 2.0} ${wheel_radius + 0.08}"/>
+    <xacro:inertial_box mass="18.0" x="${fork_length}" y="${fork_width}" z="${fork_height}">
+      <origin xyz="${mast_x + carriage_depth + fork_length / 2.0} -${fork_gap / 2.0} ${body_base_z + 0.08}"/>
     </xacro:inertial_box>
   </link>
@@ -178,4 +175,5 @@
   <link name="front_left_wheel_link">
     <visual>
+      <origin xyz="0 0 0" rpy="1.57079632679 0 0"/>
       <geometry>
         <cylinder radius="${wheel_radius}" length="${wheel_width}"/>
@@ -186,10 +184,11 @@
     </visual>
     <collision>
-      <geometry>
-        <cylinder radius="${wheel_radius}" length="${wheel_width}"/>
-      </geometry>
-    </collision>
-    <xacro:inertial_cylinder mass="45.0" length="${wheel_width}" radius="${wheel_radius}">
-      <origin xyz="0 0 0"/>
+      <origin xyz="0 0 0" rpy="1.57079632679 0 0"/>
+      <geometry>
+        <cylinder radius="${wheel_radius}" length="${wheel_width}"/>
+      </geometry>
+    </collision>
+    <xacro:inertial_cylinder mass="38.0" length="${wheel_width}" radius="${wheel_radius}">
+      <origin xyz="0 0 0" rpy="1.57079632679 0 0"/>
     </xacro:inertial_cylinder>
   </link>
@@ -197,9 +196,11 @@
     <parent link="base_link"/>
     <child link="front_left_wheel_link"/>
-    <origin xyz="${front_axle_x} ${front_track / 2.0} ${wheel_radius}" rpy="-1.57079632679 0 0"/>
-    <axis xyz="0 0 1"/>
+    <origin xyz="${front_axle_x} ${front_track / 2.0} ${wheel_radius}" rpy="0 0 0"/>
+    <axis xyz="0 1 0"/>
+    <dynamics damping="0.40" friction="0.05"/>
   </joint>
   <link name="front_right_wheel_link">
     <visual>
+      <origin xyz="0 0 0" rpy="1.57079632679 0 0"/>
       <geometry>
         <cylinder radius="${wheel_radius}" length="${wheel_width}"/>
@@ -208,10 +209,11 @@
     </visual>
     <collision>
-      <geometry>
-        <cylinder radius="${wheel_radius}" length="${wheel_width}"/>
-      </geometry>
-    </collision>
-    <xacro:inertial_cylinder mass="45.0" length="${wheel_width}" radius="${wheel_radius}">
-      <origin xyz="0 0 0"/>
+      <origin xyz="0 0 0" rpy="1.57079632679 0 0"/>
+      <geometry>
+        <cylinder radius="${wheel_radius}" length="${wheel_width}"/>
+      </geometry>
+    </collision>
+    <xacro:inertial_cylinder mass="38.0" length="${wheel_width}" radius="${wheel_radius}">
+      <origin xyz="0 0 0" rpy="1.57079632679 0 0"/>
     </xacro:inertial_cylinder>
   </link>
@@ -219,10 +221,11 @@
     <parent link="base_link"/>
     <child link="front_right_wheel_link"/>
-    <origin xyz="${front_axle_x} -${front_track / 2.0} ${wheel_radius}" rpy="1.57079632679 0 0"/>
-    <axis xyz="0 0 -1"/>
+    <origin xyz="${front_axle_x} -${front_track / 2.0} ${wheel_radius}" rpy="0 0 0"/>
+    <axis xyz="0 1 0"/>
+    <dynamics damping="0.40" friction="0.05"/>
   </joint>
   <link name="rear_left_steer_link">
     <visual>
-      <origin xyz="0 0 0.12"/>
+      <origin xyz="0 0 ${rear_steer_link_center_z}"/>
       <geometry>
         <box size="0.10 0.08 0.24"/>
@@ -230,12 +233,6 @@
       <material name="steel"/>
     </visual>
-    <collision>
-      <origin xyz="0 0 0.12"/>
-      <geometry>
-        <box size="0.10 0.08 0.24"/>
-      </geometry>
-    </collision>
-    <xacro:inertial_box mass="15.0" x="0.10" y="0.08" z="0.24">
-      <origin xyz="0 0 0.12"/>
+    <xacro:inertial_box mass="18.0" x="0.10" y="0.08" z="0.24">
+      <origin xyz="0 0 ${rear_steer_link_center_z}"/>
     </xacro:inertial_box>
   </link>
@@ -245,9 +242,10 @@
     <origin xyz="${rear_axle_x} ${rear_track / 2.0} 0.0"/>
     <axis xyz="0 0 1"/>
-    <limit lower="-0.90" upper="0.90" effort="1200.0" velocity="1.2"/>
-    <dynamics damping="15.0" friction="0.5"/>
+    <limit lower="-0.60" upper="0.60" effort="3200.0" velocity="1.2"/>
+    <dynamics damping="12.0" friction="0.4"/>
   </joint>
   <link name="rear_left_wheel_link">
     <visual>
+      <origin xyz="0 0 0" rpy="1.57079632679 0 0"/>
       <geometry>
         <cylinder radius="${wheel_radius}" length="${wheel_width}"/>
@@ -256,10 +254,11 @@
     </visual>
     <collision>
-      <geometry>
-        <cylinder radius="${wheel_radius}" length="${wheel_width}"/>
-      </geometry>
-    </collision>
-    <xacro:inertial_cylinder mass="30.0" length="${wheel_width}" radius="${wheel_radius}">
-      <origin xyz="0 0 0"/>
+      <origin xyz="0 0 0" rpy="1.57079632679 0 0"/>
+      <geometry>
+        <cylinder radius="${wheel_radius}" length="${wheel_width}"/>
+      </geometry>
+    </collision>
+    <xacro:inertial_cylinder mass="42.0" length="${wheel_width}" radius="${wheel_radius}">
+      <origin xyz="0 0 0" rpy="1.57079632679 0 0"/>
     </xacro:inertial_cylinder>
   </link>
@@ -267,11 +266,11 @@
     <parent link="rear_left_steer_link"/>
     <child link="rear_left_wheel_link"/>
-    <origin xyz="0 0 ${wheel_radius}" rpy="-1.57079632679 0 0"/>
-    <axis xyz="0 0 1"/>
-    <dynamics damping="0.2" friction="0.0"/>
+    <origin xyz="0 0 ${wheel_radius}" rpy="0 0 0"/>
+    <axis xyz="0 1 0"/>
+    <dynamics damping="0.45" friction="0.05"/>
   </joint>
   <link name="rear_right_steer_link">
     <visual>
-      <origin xyz="0 0 0.12"/>
+      <origin xyz="0 0 ${rear_steer_link_center_z}"/>
       <geometry>
         <box size="0.10 0.08 0.24"/>
@@ -279,12 +278,6 @@
       <material name="steel"/>
     </visual>
-    <collision>
-      <origin xyz="0 0 0.12"/>
-      <geometry>
-        <box size="0.10 0.08 0.24"/>
-      </geometry>
-    </collision>
-    <xacro:inertial_box mass="15.0" x="0.10" y="0.08" z="0.24">
-      <origin xyz="0 0 0.12"/>
+    <xacro:inertial_box mass="18.0" x="0.10" y="0.08" z="0.24">
+      <origin xyz="0 0 ${rear_steer_link_center_z}"/>
     </xacro:inertial_box>
   </link>
@@ -294,9 +287,10 @@
     <origin xyz="${rear_axle_x} -${rear_track / 2.0} 0.0"/>
     <axis xyz="0 0 1"/>
-    <limit lower="-0.90" upper="0.90" effort="1200.0" velocity="1.2"/>
-    <dynamics damping="15.0" friction="0.5"/>
+    <limit lower="-0.60" upper="0.60" effort="3200.0" velocity="1.2"/>
+    <dynamics damping="12.0" friction="0.4"/>
   </joint>
   <link name="rear_right_wheel_link">
     <visual>
+      <origin xyz="0 0 0" rpy="1.57079632679 0 0"/>
       <geometry>
         <cylinder radius="${wheel_radius}" length="${wheel_width}"/>
@@ -305,10 +299,11 @@
     </visual>
     <collision>
-      <geometry>
-        <cylinder radius="${wheel_radius}" length="${wheel_width}"/>
-      </geometry>
-    </collision>
-    <xacro:inertial_cylinder mass="30.0" length="${wheel_width}" radius="${wheel_radius}">
-      <origin xyz="0 0 0"/>
+      <origin xyz="0 0 0" rpy="1.57079632679 0 0"/>
+      <geometry>
+        <cylinder radius="${wheel_radius}" length="${wheel_width}"/>
+      </geometry>
+    </collision>
+    <xacro:inertial_cylinder mass="42.0" length="${wheel_width}" radius="${wheel_radius}">
+      <origin xyz="0 0 0" rpy="1.57079632679 0 0"/>
     </xacro:inertial_cylinder>
   </link>
@@ -316,13 +311,13 @@
     <parent link="rear_right_steer_link"/>
     <child link="rear_right_wheel_link"/>
-    <origin xyz="0 0 ${wheel_radius}" rpy="1.57079632679 0 0"/>
-    <axis xyz="0 0 -1"/>
-    <dynamics damping="0.2" friction="0.0"/>
+    <origin xyz="0 0 ${wheel_radius}" rpy="0 0 0"/>
+    <axis xyz="0 1 0"/>
+    <dynamics damping="0.45" friction="0.05"/>
   </joint>
   <link name="imu_link"/>
   <joint name="imu_joint" type="fixed">
-    <parent link="chassis_link"/>
+    <parent link="base_link"/>
     <child link="imu_link"/>
-    <origin xyz="0.0 0.0 ${wheel_radius + chassis_height + 0.15}"/>
+    <origin xyz="0.0 0.0 ${body_base_z + chassis_height + 0.15}"/>
   </joint>
   <link name="laser_frame_link">
@@ -352,9 +347,17 @@
     </hardware>
     <joint name="front_left_wheel_joint">
+      <state_interface name="velocity"/>
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