Commit message: Stabilize physics forklift wheel geometry

File: src/forklift_description/urdf/forklift_common.xacro (robot description, xacro)
@@ -20,5 +20,5 @@
       </collision>
       <xacro:inertial_box mass="${chassis_mass + payload_mass}" x="1.65" y="1.05" z="0.50">
-        <origin xyz="-0.08 0 0.30" rpy="0 0 0"/>
+        <origin xyz="-0.20 0 0.18" rpy="0 0 0"/>
       </xacro:inertial_box>
     </link>

File: src/forklift_description/urdf/forklift_physics.xacro (robot description, xacro)
@@ -7,8 +7,9 @@
   <xacro:arg name="enable_depth_camera" default="false"/>
   <xacro:property name="wheelbase" value="1.35"/>
-  <xacro:property name="track_width" value="1.05"/>
+  <xacro:property name="track_width" value="1.25"/>
   <xacro:property name="wheel_radius" value="0.16"/>
   <xacro:property name="wheel_width" value="0.10"/>
   <xacro:property name="wheel_mass" value="12.0"/>
+  <xacro:property name="wheel_z" value="-0.16"/>
   <xacro:property name="steer_lower" value="-0.55"/>
   <xacro:property name="steer_upper" value="0.55"/>
@@ -26,5 +27,5 @@
     x="${wheelbase * 0.5}"
     y="${track_width * 0.5}"
-    z="-0.10"
+    z="${wheel_z}"
     wheel_radius="${wheel_radius}"
     wheel_width="${wheel_width}"
@@ -35,5 +36,5 @@
     x="${wheelbase * 0.5}"
     y="${-track_width * 0.5}"
-    z="-0.10"
+    z="${wheel_z}"
     wheel_radius="${wheel_radius}"
     wheel_width="${wheel_width}"
@@ -44,5 +45,5 @@
     x="${-wheelbase * 0.5}"
     y="${track_width * 0.5}"
-    z="-0.10"
+    z="${wheel_z}"
     wheel_radius="${wheel_radius}"
     wheel_width="${wheel_width}"
@@ -56,5 +57,5 @@
     x="${-wheelbase * 0.5}"
     y="${-track_width * 0.5}"
-    z="-0.10"
+    z="${wheel_z}"
     wheel_radius="${wheel_radius}"
     wheel_width="${wheel_width}"

File: src/forklift_description/urdf/forklift_wheels.xacro (robot description, xacro)
@@ -21,5 +21,5 @@
       <axis xyz="0 0 1"/>
       <limit lower="${steering_lower}" upper="${steering_upper}" effort="80.0" velocity="${steering_velocity}"/>
-      <dynamics damping="2.0" friction="0.2"/>
+      <dynamics damping="8.0" friction="1.0"/>
     </joint>
     <link name="${prefix}_wheel_link">
@@ -42,13 +42,13 @@
       <origin xyz="0 0 0" rpy="0 0 0"/>
       <axis xyz="0 1 0"/>
-      <dynamics damping="0.08" friction="0.02"/>
+      <dynamics damping="0.5" friction="0.2"/>
     </joint>
     <gazebo reference="${prefix}_wheel_link">
       <mu1>0.9</mu1>
       <mu2>0.65</mu2>
-      <kp>800000.0</kp>
-      <kd>20.0</kd>
-      <minDepth>0.001</minDepth>
-      <maxVel>0.2</maxVel>
+      <kp>250000.0</kp>
+      <kd>80.0</kd>
+      <minDepth>0.0005</minDepth>
+      <maxVel>0.05</maxVel>
     </gazebo>
   </xacro:macro>
@@ -73,13 +73,13 @@
       <origin xyz="${x} ${y} ${z}" rpy="0 0 0"/>
       <axis xyz="0 1 0"/>
-      <dynamics damping="0.08" friction="0.02"/>
+      <dynamics damping="0.5" friction="0.2"/>
     </joint>
     <gazebo reference="${prefix}_wheel_link">
       <mu1>0.9</mu1>
       <mu2>0.65</mu2>
-      <kp>800000.0</kp>
-      <kd>20.0</kd>
-      <minDepth>0.001</minDepth>
-      <maxVel>0.2</maxVel>
+      <kp>250000.0</kp>
+      <kd>80.0</kd>
+      <minDepth>0.0005</minDepth>
+      <maxVel>0.05</maxVel>
     </gazebo>
   </xacro:macro>

Commit message: Rebase physics model around wheel center height

File: src/forklift_description/urdf/forklift_common.xacro (robot description, xacro)
@@ -7,18 +7,18 @@
       <parent link="base_footprint"/>
       <child link="${base_link}"/>
-      <origin xyz="0 0 0.18" rpy="0 0 0"/>
+      <origin xyz="0 0 0.16" rpy="0 0 0"/>
     </joint>
     <link name="${base_link}">
       <visual>
-        <origin xyz="0 0 0.25" rpy="0 0 0"/>
-        <geometry><box size="1.65 1.05 0.50"/></geometry>
+        <origin xyz="0 0 0.30" rpy="0 0 0"/>
+        <geometry><box size="1.65 1.05 0.36"/></geometry>
         <material name="green"><color rgba="0.1 0.8 0.2 1.0"/></material>
       </visual>
       <collision>
-        <origin xyz="0 0 0.25" rpy="0 0 0"/>
-        <geometry><box size="1.65 1.05 0.50"/></geometry>
+        <origin xyz="0 0 0.30" rpy="0 0 0"/>
+        <geometry><box size="1.65 1.05 0.36"/></geometry>
       </collision>
-      <xacro:inertial_box mass="${chassis_mass + payload_mass}" x="1.65" y="1.05" z="0.50">
-        <origin xyz="-0.20 0 0.18" rpy="0 0 0"/>
+      <xacro:inertial_box mass="${chassis_mass + payload_mass}" x="1.65" y="1.05" z="0.36">
+        <origin xyz="-0.28 0 0.22" rpy="0 0 0"/>
       </xacro:inertial_box>
     </link>
@@ -40,5 +40,5 @@
       <parent link="${base_link}"/>
       <child link="mast_link"/>
-      <origin xyz="0.78 0 0.42" rpy="0 0 0"/>
+      <origin xyz="0.72 0 0.36" rpy="0 0 0"/>
     </joint>
     <link name="fork_carriage_link">

File: src/forklift_description/urdf/forklift_physics.xacro (robot description, xacro)
@@ -11,5 +11,5 @@
   <xacro:property name="wheel_width" value="0.10"/>
   <xacro:property name="wheel_mass" value="12.0"/>
-  <xacro:property name="wheel_z" value="-0.16"/>
+  <xacro:property name="wheel_z" value="0.0"/>
   <xacro:property name="steer_lower" value="-0.55"/>
   <xacro:property name="steer_upper" value="0.55"/>
@@ -68,6 +68,6 @@
     <mu1>0.85</mu1>
     <mu2>0.65</mu2>
-    <kp>900000.0</kp>
-    <kd>25.0</kd>
+    <kp>250000.0</kp>
+    <kd>80.0</kd>
   </gazebo>
 </robot>

File: src/forklift_description/urdf/forklift_wheels.xacro (robot description, xacro)
@@ -47,4 +47,5 @@
       <mu1>0.9</mu1>
       <mu2>0.65</mu2>
+      <fdir1>1 0 0</fdir1>
       <kp>250000.0</kp>
       <kd>80.0</kd>
@@ -78,4 +79,5 @@
       <mu1>0.9</mu1>
       <mu2>0.65</mu2>
+      <fdir1>1 0 0</fdir1>
       <kp>250000.0</kp>
       <kd>80.0</kd>

Commit message: Rework physics URDF wheel mounting geometry

File: src/forklift_description/urdf/forklift_common.xacro (robot description, xacro)
@@ -3,36 +3,36 @@
   <xacro:include filename="forklift_inertials.xacro"/>
   <xacro:macro name="forklift_common_body" params="base_link:=base_link chassis_mass:=850.0 payload_mass:=0.0 enable_depth_camera:=true">
-    <link name="base_footprint"/>
-    <joint name="base_footprint_joint" type="fixed">
-      <parent link="base_footprint"/>
-      <child link="${base_link}"/>
-      <origin xyz="0 0 0.16" rpy="0 0 0"/>
-    </joint>
     <link name="${base_link}">
       <visual>
-        <origin xyz="0 0 0.30" rpy="0 0 0"/>
-        <geometry><box size="1.65 1.05 0.36"/></geometry>
+        <origin xyz="-0.04 0 0.24" rpy="0 0 0"/>
+        <geometry><box size="1.58 0.92 0.32"/></geometry>
         <material name="green"><color rgba="0.1 0.8 0.2 1.0"/></material>
       </visual>
       <collision>
-        <origin xyz="0 0 0.30" rpy="0 0 0"/>
-        <geometry><box size="1.65 1.05 0.36"/></geometry>
+        <origin xyz="-0.04 0 0.24" rpy="0 0 0"/>
+        <geometry><box size="1.58 0.92 0.32"/></geometry>
       </collision>
-      <xacro:inertial_box mass="${chassis_mass + payload_mass}" x="1.65" y="1.05" z="0.36">
-        <origin xyz="-0.28 0 0.22" rpy="0 0 0"/>
+      <xacro:inertial_box mass="${chassis_mass + payload_mass}" x="1.58" y="0.92" z="0.32">
+        <origin xyz="-0.26 0 0.18" rpy="0 0 0"/>
       </xacro:inertial_box>
     </link>
+    <link name="base_footprint"/>
+    <joint name="base_footprint_joint" type="fixed">
+      <parent link="${base_link}"/>
+      <child link="base_footprint"/>
+      <origin xyz="0 0 -0.16" rpy="0 0 0"/>
+    </joint>
     <link name="mast_link">
       <visual>
-        <origin xyz="0 0 0.9" rpy="0 0 0"/>
-        <geometry><box size="0.16 1.0 1.8"/></geometry>
+        <origin xyz="0 0 0.74" rpy="0 0 0"/>
+        <geometry><box size="0.16 0.92 1.48"/></geometry>
         <material name="red"><color rgba="0.9 0.1 0.1 1.0"/></material>
       </visual>
       <collision>
-        <origin xyz="0 0 0.9" rpy="0 0 0"/>
-        <geometry><box size="0.16 1.0 1.8"/></geometry>
+        <origin xyz="0 0 0.74" rpy="0 0 0"/>
+        <geometry><box size="0.16 0.92 1.48"/></geometry>
       </collision>
-      <xacro:inertial_box mass="90.0" x="0.16" y="1.0" z="1.8">
-        <origin xyz="0 0 0.9" rpy="0 0 0"/>
+      <xacro:inertial_box mass="55.0" x="0.16" y="0.92" z="1.48">
+        <origin xyz="0 0 0.58" rpy="0 0 0"/>
       </xacro:inertial_box>
     </link>
@@ -40,5 +40,5 @@
       <parent link="${base_link}"/>
       <child link="mast_link"/>
-      <origin xyz="0.72 0 0.36" rpy="0 0 0"/>
+      <origin xyz="0.70 0 0.34" rpy="0 0 0"/>
     </joint>
     <link name="fork_carriage_link">
@@ -58,5 +58,5 @@
       <parent link="mast_link"/>
       <child link="fork_carriage_link"/>
-      <origin xyz="0.08 0 0.15" rpy="0 0 0"/>
+      <origin xyz="0.08 0 -0.20" rpy="0 0 0"/>
       <axis xyz="0 0 1"/>
       <limit lower="0.0" upper="0.8" effort="1000.0" velocity="0.25"/>
@@ -71,5 +71,5 @@
       <parent link="fork_carriage_link"/>
       <child link="left_fork_link"/>
-      <origin xyz="0.08 0.32 -0.10" rpy="0 0 0"/>
+      <origin xyz="0.08 0.32 -0.16" rpy="0 0 0"/>
     </joint>
     <link name="right_fork_link">
@@ -81,5 +81,5 @@
       <parent link="fork_carriage_link"/>
       <child link="right_fork_link"/>
-      <origin xyz="0.08 -0.32 -0.10" rpy="0 0 0"/>
+      <origin xyz="0.08 -0.32 -0.16" rpy="0 0 0"/>
     </joint>
     <link name="laser_frame_link">

File: src/forklift_description/urdf/forklift_wheels.xacro (robot description, xacro)
@@ -5,11 +5,11 @@
       <visual>
         <origin xyz="0 0 0" rpy="0 0 0"/>
-        <geometry><box size="0.12 0.08 0.10"/></geometry>
+        <geometry><box size="0.12 0.14 0.18"/></geometry>
         <material name="dark_gray"><color rgba="0.05 0.05 0.05 1.0"/></material>
       </visual>
       <collision>
-        <geometry><box size="0.12 0.08 0.10"/></geometry>
+        <geometry><box size="0.12 0.14 0.18"/></geometry>
       </collision>
-      <xacro:inertial_box mass="2.0" x="0.12" y="0.08" z="0.10">
+      <xacro:inertial_box mass="3.0" x="0.12" y="0.14" z="0.18">
         <origin xyz="0 0 0" rpy="0 0 0"/>
       </xacro:inertial_box>
@@ -55,4 +55,22 @@
   </xacro:macro>
   <xacro:macro name="fixed_wheel" params="prefix parent x y z wheel_radius wheel_width wheel_mass">
+    <link name="${prefix}_wheel_mount_link">
+      <visual>
+        <origin xyz="0 0 0" rpy="0 0 0"/>
+        <geometry><box size="0.14 0.14 0.16"/></geometry>
+        <material name="dark_gray"><color rgba="0.05 0.05 0.05 1.0"/></material>
+      </visual>
+      <collision>
+        <geometry><box size="0.14 0.14 0.16"/></geometry>
+      </collision>
+      <xacro:inertial_box mass="3.0" x="0.14" y="0.14" z="0.16">
+        <origin xyz="0 0 0" rpy="0 0 0"/>
+      </xacro:inertial_box>
+    </link>
+    <joint name="${prefix}_wheel_mount_joint" type="fixed">
+      <parent link="${parent}"/>
+      <child link="${prefix}_wheel_mount_link"/>
+      <origin xyz="${x} ${y} ${z}" rpy="0 0 0"/>
+    </joint>
     <link name="${prefix}_wheel_link">
       <visual>
@@ -70,7 +88,7 @@
     </link>
     <joint name="${prefix}_wheel_rotation_joint" type="continuous">
-      <parent link="${parent}"/>
+      <parent link="${prefix}_wheel_mount_link"/>
       <child link="${prefix}_wheel_link"/>
-      <origin xyz="${x} ${y} ${z}" rpy="0 0 0"/>
+      <origin xyz="0 0 0" rpy="0 0 0"/>
       <axis xyz="0 1 0"/>
       <dynamics damping="0.5" friction="0.2"/>
